File: LightListener/LightListener.kicad_pcb (KiCad board)
At the start: 2 copper layers, 22 parts, among them J1 AudioJack3_SwitchTR, J2 Conn_01x01, J3 Conn_01x01, Q1 Q_Photo_NPN, Q2 Q_Photo_NPN

Commit message: PCB design (brief)
Parts:
- added H1: MountingHole_Pad, MountingHole:MountingHole_3.2mm_M3_Pad_Via, F.Cu at (196.0, 87.0)
- added H2: MountingHole_Pad, MountingHole:MountingHole_3.2mm_M3_Pad_Via, F.Cu at (211.0, 87.0)
- C5, C6, C7: value 470uF -> 100uF; footprint Capacitor_SMD:CP_Elec_8x11.9 -> Capacitor_SMD:C_1206_3216Metric
- U2: value ~ -> TDA2822G-S08; footprint Package_DIP:DIP-8_W7.62mm_LongPads -> Package_SO:SOP-8_3.9x4.9mm_P1.27mm
- moved J1 102.2 mm to (211.0, 135.0), turned to 180 degrees
- moved R1 93.7 mm to (200.7, 41.5), turned to 180 degrees
- moved R3 87.9 mm to (206.2, 41.5)
- moved C2 87.3 mm to (206.2, 44.8), turned to 180 degrees
- moved U1 86.1 mm to (192.5, 130.0), turned to 90 degrees
- moved C1 82.2 mm to (200.7, 44.8)
- moved J2 79.4 mm to (212.0, 109.5), turned to 90 degrees
- moved J3 73.5 mm to (212.0, 103.0), turned to 90 degrees
- moved Q2 69.5 mm to (212.5, 45.3), turned to 135 degrees
- moved C7 65.5 mm to (214.3, 115.2)
- moved Q1 63.9 mm to (196.0, 43.5), turned to -135 degrees
- moved C6 60.0 mm to (208.2, 115.2)
- moved C9 57.2 mm to (214.3, 118.8)
- moved R6 53.2 mm to (214.3, 121.5), turned to 180 degrees
- moved C8 51.1 mm to (208.2, 118.8)
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Routing:
- net GND: track 0.00 -> 238.6 mm, vias 0 -> 11
- net VCC: track 0.00 -> 113.5 mm
- net Net-(C2-Pad2): track 0.00 -> 84.5 mm
- net Net-(C1-Pad2): track 0.00 -> 78.8 mm
- net Net-(J2-Pin_1): track 0.00 -> 26.7 mm, vias 0 -> 1
- net Net-(U2-OUT2): track 0.00 -> 20.6 mm, vias 0 -> 2
- net Net-(U2-IN2): track 0.00 -> 17.9 mm
- net Net-(U2-IN1): track 0.00 -> 14.6 mm
- net Net-(U2-OUT1): track 0.00 -> 14.1 mm, vias 0 -> 2
- net Net-(C6-Pad2): track 0.00 -> 13.8 mm
- net Net-(C7-Pad2): track 0.00 -> 13.2 mm
- net Net-(Q2-C): track 0.00 -> 9.27 mm
- net Net-(Q1-C): track 0.00 -> 7.76 mm
- net Net-(R2-Pad2): track 0.00 -> 6.02 mm
- net Net-(R4-Pad2): track 0.00 -> 4.78 mm
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- added copper zone on B.Cu, net GND
- added copper zone on F.Cu, net GND
Other:
- board outline added: 29 x 96 mm

Commit message: transmitter pcb design
Parts:
- moved H1 44.6 mm to (203.5, 43.0)
- moved H2 19.5 mm to (203.5, 105.0)
- moved Q1 14.8 mm to (210.8, 43.2)
- moved Q2 14.5 mm to (198.0, 45.0)
- moved R1 13.6 mm to (214.0, 44.0)
- moved R3 13.4 mm to (193.0, 44.0)
- moved C1 13.3 mm to (214.0, 46.0)
- moved C2 13.3 mm to (193.0, 46.0)
- moved J2 0.50 mm to (212.5, 109.5)
- moved J3 0.50 mm to (212.5, 103.0)
Routing:
- net GND: track 238.6 -> 192.1 mm, vias 11 -> 37
- net VCC: track 113.5 -> 126.3 mm, vias 0 -> 2
- net Net-(C1-Pad2): track 78.8 -> 89.0 mm, vias 0 -> 2
- net Net-(C2-Pad2): track 84.5 -> 88.0 mm
- net Net-(Q1-C): track 7.76 -> 4.73 mm
- net Net-(Q2-C): track 9.27 -> 6.61 mm
Other:
- board size 29 x 96 mm -> 29 x 99 mm
- board text added: "9V"
- board text added: "GND"
- board text added: "Stereo Light Receiver"
- board text added: "for OPEN HOME OPEN STUDIO HORIO KANTA v1.0 / 2024-03-26"
