File: LightListener/LightListener.kicad_sch (KiCad schematic)
At the start: 22 parts, among them J1 AudioJack3_SwitchTR, J2 Conn_01x01, J3 Conn_01x01, Q1 Q_Photo_NPN, Q2 Q_Photo_NPN

Commit message: PCB design (brief)
Parts:
- removed C5, C6, C7: 470uF, Capacitor_SMD:CP_Elec_8x11.9, symbol Device:C_Polarized
- added C5, C6, C7: 100uF, Capacitor_SMD:C_1206_3216Metric, symbol Device:C
- added H1, H2: MountingHole_Pad, MountingHole:MountingHole_3.2mm_M3_Pad_Via, symbol Mechanical:MountingHole_Pad
- U2: value ~ -> TDA2822G-S08; footprint Package_DIP:DIP-8_W7.62mm_LongPads -> Package_SO:SOP-8_3.9x4.9mm_P1.27mm
Connections:
- net GND: now also C5.2, H1.1, H2.1
- net VCC: now also C5.1
- net at C8.2, J1.T: now also C6.2
- net at C9.2, J1.R: now also C7.2
- net at U2.3 (OUT2): now also C7.1
- net at U2.1 (OUT1): now also C6.1
Changed lines of the file:
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@@
+    )
+  )
+  (symbol (lib_id "power:GND") (at 144.78 55.88 0) (unit 1)
+    (in_bom yes) (on_board yes) (dnp no) (fields_autoplaced)
+    (property "Reference" "#PWR015" (at 144.78 62.23 0)
+      (effects (font (size 1.27 1.27)) hide)
+    )
+    (property "Value" "GND" (at 144.78 60.96 0)
+      (effects (font (size 1.27 1.27)))
+    )
+    (property "Footprint" "" (at 144.78 55.88 0)
+      (effects (font (size 1.27 1.27)) hide)
+    )
+    (property "Datasheet" "" (at 144.78 55.88 0)
+      (effects (font (size 1.27 1.27)) hide)
+    )
+    (pin "1")
+    (instances
+      (project "LightListener"
+        (path "/ad39a340-bbfc-48e0-8c8a-e66de62c709c"
+          (reference "#PWR015") (unit 1)
+        )
+      )
     )
   )
@@
     )
   )
+  (symbol (lib_id "Mechanical:MountingHole_Pad") (at 144.78 69.85 0) (unit 1)
+    (in_bom yes) (on_board yes) (dnp no) (fields_autoplaced)
+    (property "Reference" "H2" (at 147.32 67.31 0)
+      (effects (font (size 1.27 1.27)) (justify left))
+    )
+    (property "Value" "MountingHole_Pad" (at 147.32 69.85 0)
+      (effects (font (size 1.27 1.27)) (justify left))
+    )
+    (property "Footprint" "MountingHole:MountingHole_3.2mm_M3_Pad_Via" (at 144.78 69.85 0)
+      (effects (font (size 1.27 1.27)) hide)
+    )
+    (property "Datasheet" "~" (at 144.78 69.85 0)
+      (effects (font (size 1.27 1.27)) hide)
+    )
+    (pin "1")
+    (instances
+      (project "LightListener"
+        (path "/ad39a340-bbfc-48e0-8c8a-e66de62c709c"
+          (reference "H2") (unit 1)
+        )
+      )
+    )
+  )
   (symbol (lib_id "power:GND") (at 99.06 139.7 0) (unit 1)
     (in_bom yes) (on_board yes) (dnp no) (fields_autoplaced)
@@
         (path "/ad39a340-bbfc-48e0-8c8a-e66de62c709c"
           (reference "#PWR05") (unit 1)
+        )
+      )
+    )
+  )
+  (symbol (lib_id "Device:C") (at 104.14 106.68 0) (unit 1)
+    (in_bom yes) (on_board yes) (dnp no) (fields_autoplaced)
+    (property "Reference" "C5" (at 107.95 105.41 0)
+      (effects (font (size 1.27 1.27)) (justify left))
+    )
+    (property "Value" "100uF" (at 107.95 107.95 0)
+      (effects (font (size 1.27 1.27)) (justify left))
+    )
+    (property "Footprint" "Capacitor_SMD:C_1206_3216Metric" (at 105.1052 110.49 0)
+      (effects (font (size 1.27 1.27)) hide)
+    )
+    (property "Datasheet" "~" (at 104.14 106.68 0)
+      (effects (font (size 1.27 1.27)) hide)
+    )
+    (pin "1")
+    (pin "2")
+    (instances
+      (project "LightListener"
+        (path "/ad39a340-bbfc-48e0-8c8a-e66de62c709c"
+          (reference "C5") (unit 1)
         )
       )
@@
     )
   )
-  (symbol (lib_id "Device:C_Polarized") (at 132.08 124.46 90) (unit 1)
-    (in_bom yes) (on_board yes) (dnp no) (fields_autoplaced)
-    (property "Reference" "C7" (at 131.191 116.84 90)
-      (effects (font (size 1.27 1.27)))
-    )
-    (property "Value" "470uF" (at 131.191 119.38 90)
-      (effects (font (size 1.27 1.27)))
-    )
-    (property "Footprint" "Capacitor_SMD:CP_Elec_8x11.9" (at 135.89 123.4948 0)
-      (effects (font (size 1.27 1.27)) hide)
-    )
-    (property "Datasheet" "~" (at 132.08 124.46 0)
-      (effects (font (size 1.27 1.27)) hide)
-    )
-    (pin "1")
-    (pin "2")
-    (instances
-      (project "LightListener"
-        (path "/ad39a340-bbfc-48e0-8c8a-e66de62c709c"
-          (reference "C7") (unit 1)
-        )
-      )
-    )
-  )
-  (symbol (lib_id "Device:C_Polarized") (at 104.14 106.68 0) (unit 1)
-    (in_bom yes) (on_board yes) (dnp no) (fields_autoplaced)
-    (property "Reference" "C5" (at 107.95 104.521 0)
-      (effects (font (size 1.27 1.27)) (justify left))
-    )
-    (property "Value" "470uF" (at 107.95 107.061 0)
-      (effects (font (size 1.27 1.27)) (justify left))
-    )
-    (property "Footprint" "Capacitor_SMD:CP_Elec_8x11.9" (at 105.1052 110.49 0)
-      (effects (font (size 1.27 1.27)) hide)
-    )
-    (property "Datasheet" "~" (at 104.14 106.68 0)
-      (effects (font (size 1.27 1.27)) hide)
-    )
-    (pin "1")
-    (pin "2")
-    (instances
-      (project "LightListener"
-        (path "/ad39a340-bbfc-48e0-8c8a-e66de62c709c"
-          (reference "C5") (unit 1)
+  (symbol (lib_id "Device:C") (at 132.08 113.03 90) (unit 1)
+    (in_bom yes) (on_board yes) (dnp no) (fields_autoplaced)
+    (property "Reference" "C6" (at 132.08 105.41 90)
+      (effects (font (size 1.27 1.27)))
+    )
+    (property "Value" "100uF" (at 132.08 107.95 90)
+      (effects (font (size 1.27 1.27)))
+    )
+    (property "Footprint" "Capacitor_SMD:C_1206_3216Metric" (at 135.89 112.0648 0)
+      (effects (font (size 1.27 1.27)) hide)
+    )
+    (property "Datasheet" "~" (at 132.08 113.03 0)
+      (effects (font (size 1.27 1.27)) hide)
+    )
+    (pin "1")
+    (pin "2")
+    (instances
+      (project "LightListener"
+        (path "/ad39a340-bbfc-48e0-8c8a-e66de62c709c"
+          (reference "C6") (unit 1)
         )
       )
@@
     )
   )
-  (symbol (lib_id "Device:C_Polarized") (at 132.08 113.03 90) (unit 1)
-    (in_bom yes) (on_board yes) (dnp no) (fields_autoplaced)
-    (property "Reference" "C6" (at 131.191 105.41 90)
-      (effects (font (size 1.27 1.27)))
-    )
-    (property "Value" "470uF" (at 131.191 107.95 90)
-      (effects (font (size 1.27 1.27)))
-    )
-    (property "Footprint" "Capacitor_SMD:CP_Elec_8x11.9" (at 135.89 112.0648 0)
-      (effects (font (size 1.27 1.27)) hide)
-    )
-    (property "Datasheet" "~" (at 132.08 113.03 0)
-      (effects (font (size 1.27 1.27)) hide)
-    )
-    (pin "1")
-    (pin "2")
-    (instances
-      (project "LightListener"
-        (path "/ad39a340-bbfc-48e0-8c8a-e66de62c709c"
-          (reference "C6") (unit 1)
-        )
-      )
-    )
-  )
   (symbol (lib_id "Local_Library:TDA2822") (at 116.84 119.38 0) (unit 1)
     (in_bom yes) (on_board yes) (dnp no) (fields_autoplaced)
@@
       (effects (font (size 1.27 1.27)) (justify left))
     )
-    (property "Value" "~" (at 116.84 119.38 0)
-      (effects (font (size 1.27 1.27)))
-    )
-    (property "Footprint" "Package_DIP:DIP-8_W7.62mm_LongPads" (at 116.84 119.38 0)
+    (property "Value" "TDA2822G-S08" (at 116.84 119.38 0)
+      (effects (font (size 1.27 1.27)))
+    )
+    (property "Footprint" "Package_SO:SOP-8_3.9x4.9mm_P1.27mm" (at 116.84 119.38 0)
       (effects (font (size 1.27 1.27)) hide)
     )
@@
     )
   )
+  (symbol (lib_id "power:GND") (at 144.78 72.39 0) (unit 1)
+    (in_bom yes) (on_board yes) (dnp no) (fields_autoplaced)
+    (property "Reference" "#PWR016" (at 144.78 78.74 0)
+      (effects (font (size 1.27 1.27)) hide)
+    )
+    (property "Value" "GND" (at 144.78 77.47 0)
+      (effects (font (size 1.27 1.27)))
+    )
+    (property "Footprint" "" (at 144.78 72.39 0)
+      (effects (font (size 1.27 1.27)) hide)
+    )
+    (property "Datasheet" "" (at 144.78 72.39 0)
+      (effects (font (size 1.27 1.27)) hide)
+    )
+    (pin "1")
+    (instances
+      (project "LightListener"
+        (path "/ad39a340-bbfc-48e0-8c8a-e66de62c709c"
+          (reference "#PWR016") (unit 1)
+        )
+      )
+    )
+  )
   (symbol (lib_id "Device:C") (at 62.23 63.5 90) (unit 1)
     (in_bom yes) (on_board yes) (dnp no) (fields_autoplaced)
@@
         )
       )
+    )
+  )
+  (symbol (lib_id "Device:C") (at 132.08 124.46 90) (unit 1)
+    (in_bom yes) (on_board yes) (dnp no) (fields_autoplaced)
+    (property "Reference" "C7" (at 132.08 116.84 90)
+      (effects (font (size 1.27 1.27)))
+    )
+    (property "Value" "100uF" (at 132.08 119.38 90)
+      (effects (font (size 1.27 1.27)))
+    )
+    (property "Footprint" "Capacitor_SMD:C_1206_3216Metric" (at 135.89 123.4948 0)
+      (effects (font (size 1.27 1.27)) hide)
+    )
+    (property "Datasheet" "~" (at 132.08 124.46 0)
+      (effects (font (size 1.27 1.27)) hide)
+    )
+    (pin "1")
+    (pin "2")
+    (instances
+      (project "LightListener"
+        (path "/ad39a340-bbfc-48e0-8c8a-e66de62c709c"
+          (reference "C7") (unit 1)
+        )
+      )
+    )
+  )
+  (symbol (lib_id "Mechanical:MountingHole_Pad") (at 144.78 53.34 0) (unit 1)
+    (in_bom yes) (on_board yes) (dnp no) (fields_autoplaced)
+    (property "Reference" "H1" (at 147.32 50.8 0)
+      (effects (font (size 1.27 1.27)) (justify left))
+    )
+    (property "Value" "MountingHole_Pad" (at 147.32 53.34 0)
+      (effects (font (size 1.27 1.27)) (justify left))
+    )
+    (property "Footprint" "MountingHole:MountingHole_3.2mm_M3_Pad_Via" (at 144.78 53.34 0)
+      (effects (font (size 1.27 1.27)) hide)
+    )
+    (property "Datasheet" "~" (at 144.78 53.34 0)
+      (effects (font (size 1.27 1.27)) hide)
+    )
+    (pin "1")
+    (instances
+      (project "LightListener"
+        (path "/ad39a340-bbfc-48e0-8c8a-e66de62c709c"
+          (reference "H1") (unit 1)
+        )
+      )

Commit message: Changed some resistance and capacitance values
Parts:
- C1, C2: value 47nF -> 100nF
- R2, R4: value 100k -> 10k
- U1: value ~ -> 10k
Changed lines of the file:
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@@
 			)
 		)
-		(property "Value" "47nF"
+		(property "Value" "100nF"
 			(at 62.23 101.6 90)
 			(effects
@@
 			)
 		)
-		(property "Value" "~"
+		(property "Value" "10k"
 			(at 88.9 91.44 0)
 			(effects
@@
 			)
 		)
-		(property "Value" "47nF"
+		(property "Value" "100nF"
 			(at 62.23 58.42 90)
 			(effects
@@
 		(fields_autoplaced yes)
 		(property "Reference" "R4"
-			(at 72.39 101.6 0)
+			(at 72.39 101.5999 0)
 			(effects
 				(font
@@
 			)
 		)
-		(property "Value" "100k"
-			(at 72.39 104.14 0)
+		(property "Value" "10k"
+			(at 72.39 104.1399 0)
 			(effects
 				(font
@@
 		(fields_autoplaced yes)
 		(property "Reference" "R2"
-			(at 74.93 66.04 0)
+			(at 74.93 66.0399 0)
 			(effects
 				(font
@@
 			)
 		)
-		(property "Value" "100k"
-			(at 74.93 68.58 0)
-			(effects
-				(font
+		(property "Value" "10k"
+			(at 74.93 68.5799 0)
+			(effects
+				(font

Commit message: Organize schematics.
Parts:
- J1: value AudioJack3_SwitchTR -> MJ-495A
- Q1, Q2: value Q_Photo_NPN -> L-31ROPT1C
Changed lines of the file:
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@@
 			)
 		)
-		(property "Value" "AudioJack3_SwitchTR"
+		(property "Value" "MJ-495A"
 			(at 198.12 118.745 0)
 			(effects
@@
 			)
 		)
-		(property "Value" "Q_Photo_NPN"
+		(property "Value" "L-31ROPT1C"
 			(at 54.61 71.6407 0)
 			(effects
@@
 			)
 		)
-		(property "Value" "Q_Photo_NPN"
+		(property "Value" "L-31ROPT1C"
 			(at 54.61 114.8207 0)
 			(effects
